Commit message: Sync port to current robot-matching version; genericize maintainer + scrub mission-code refs
- motiond, shims, ros2_ws packages, tests, README updated to the version running on hardware
- maintainer identity -> generic; internal mission-code references removed (shareable build)

File: ros2_ws/src/ainex_gazebo/urdf/ainex.xacro (robot description, xacro)
@@ -4,3 +4,12 @@
     <xacro:include filename="$(find ainex_gazebo)/urdf/ainex.urdf.xacro"/>
     <xacro:include filename="$(find ainex_gazebo)/urdf/gazebo.xacro" />
+    <!-- VISUALIZATION PIN: fix the body to the world at standing height so the twin
+         shows a standing robot (no balance controller in sim). All servo joints
+         remain free, so driving them still animates the robot. -->
+    <link name="world"/>
+    <joint name="world_to_base" type="fixed">
+        <parent link="world"/>
+        <child link="base_link"/>
+        <origin xyz="0 0 0.33" rpy="0 0 0"/>
+    </joint>
 </robot>
